File: pcb/inside/belso_belepteto.kicad_sch (KiCad schematic)
At the start: 29 parts, among them J1 RJ12, J2 Conn_01x06_Socket, Q1 IRF7103, SW1 SW_Push, U1 MP2348GTL-P

Commit message: Schematic repair1
Connections:
- net in1 is gone; now on net In1: R4.1
- net +12V: now also U2.2 (Vin+), U2.3 (Vin+); no longer U2. (Vout-)
- net +5V: now also U2.7 (Vout+), U2.8 (Vout+); no longer U2. (Vout-)
- net GND: now also U2.4 (Vin-), U2.5 (Vout-), U2.6 (Vout-); no longer U2. (Vout-)
- net at R10.2: now also U2.1 (EN); no longer U2. (Vout-)
- net in2 renamed In2
